Commit message: lazy message, lidar, camera, drive, imu working with launch scripts

File: catkin_ws/src/proj1robot_description/urdf/proj1robot.urdf (robot description, URDF)
Before this commit: robot proj1robot, 2 links, 1 joints
Links:
- added link camera_link; visual box size=0.05 0.05 0.05
- added link imu_link; visual box size=0.05 0.025 0.02
- added link laser_link; visual cylinder length=0.02 radius=0.01
Joints:
- added joint base_link_camera: type fixed, parent base_link, child camera_link, origin xyz=0 0.35 0.225 rpy=0 0 1.5708
- added joint base_link_imu: type fixed, parent base_link, child imu_link, origin xyz=0 0.2 0.2 rpy=0 0 0
- added joint base_link_laser: type fixed, parent base_link, child laser_link, origin xyz=0 0.2 0.22 rpy=0 0 1.5708, axis 0 1 0

Commit message: all sensors available and in launch scripts

File: catkin_ws/src/proj1robot_description/urdf/proj1robot.urdf (robot description, URDF)
Before this commit: robot proj1robot, 5 links, 4 joints
Links:
- link base_link: geometry collision box size=0.2 0.4 0.2; collision box size=0.21 0.41 0.1
